File: Bottom LEDs.kicad_sch (KiCad schematic)
At the start: 28 parts

Commit message: Progress commit. Added MCU + IMU.
Connections:
- net SW7: now reaches D42.1
- net SW7: now also D41.1, D43.1, D44.1, D45.1, D46.1
- net SW9: now reaches D53.1
- net SW9: now also D54.1, D55.1, D56.1
- net SW6: now reaches D40.1
- net SW6: now also D35.1, D36.1, D37.1, D38.1, D39.1
- net SW5: now reaches D29.1
- net SW5: now also D30.1, D31.1, D32.1, D33.1, D34.1
- net SW8: now reaches D47.1
- net SW8: now also D48.1, D49.1, D50.1, D51.1, D52.1
Other:
- moved on the sheet: D53, D54, D55, D56
