File: SWD.kicad_sch (KiCad schematic)
At the start: 1 part, among them J3 009159010061911

Commit message: Re-annotated entire schematic.
Other:
- title: (none) -> Hourglass
Changed lines of the file:
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@@
 	(generator_version "9.0")
 	(paper "A4")
+	(title_block
+		(title "Hourglass")
+		(date "2025-04-23")
+		(rev "01")
+	)
 	(text "T_xxx, T is for target"
 		(exclude_from_sim yes)
@@
 		(dnp no)
 		(fields_autoplaced yes)
-		(property "Reference" "#PWR49"
+		(property "Reference" "#PWR051"
 			(at 139.7 80.01 0)
 			(effects
@@
 			(project ""
 				(path "/a75630d2-15a7-42bc-8ce0-7846cbd1da6b/25e9d76d-c367-402f-ab3d-2b63d490a5ac"
-					(reference "#PWR49")
+					(reference "#PWR051")
 					(unit 1)
 				)
@@
 		(dnp no)
 		(fields_autoplaced yes)
-		(property "Reference" "#PWR50"
+		(property "Reference" "#PWR052"
 			(at 140.97 118.11 0)
 			(effects
@@
 			(project ""
 				(path "/a75630d2-15a7-42bc-8ce0-7846cbd1da6b/25e9d76d-c367-402f-ab3d-2b63d490a5ac"
-					(reference "#PWR50")
+					(reference "#PWR052")
 					(unit 1)
 				)
