File: USB-C.kicad_sch (KiCad schematic)
At the start: 3 parts, among them J2 UJ31-CH-G2-SMT-TR

Commit message: First complete schematic with TPs.
Parts:
- renumbered R6 to R15, R7 to R16
Changed lines of the file:
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@@
 		(dnp no)
 		(fields_autoplaced yes)
-		(property "Reference" "#PWR17"
+		(property "Reference" "#PWR048"
 			(at 171.45 137.16 0)
 			(effects
@@
 			(project ""
 				(path "/a75630d2-15a7-42bc-8ce0-7846cbd1da6b/b64ac316-366b-4dad-aacf-d60ea5acbc88/d02d7f80-2025-419a-a5a1-91ce46aa8a95"
-					(reference "#PWR17")
+					(reference "#PWR048")
 					(unit 1)
 				)
@@
 		(dnp no)
 		(fields_autoplaced yes)
-		(property "Reference" "#PWR16"
+		(property "Reference" "#PWR047"
 			(at 152.4 137.16 0)
 			(effects
@@
 			(project ""
 				(path "/a75630d2-15a7-42bc-8ce0-7846cbd1da6b/b64ac316-366b-4dad-aacf-d60ea5acbc88/d02d7f80-2025-419a-a5a1-91ce46aa8a95"
-					(reference "#PWR16")
+					(reference "#PWR047")
 					(unit 1)
 				)
@@
 		(dnp no)
 		(fields_autoplaced yes)
-		(property "Reference" "R6"
+		(property "Reference" "R15"
 			(at 170.18 106.6798 90)
 			(effects
@@
 			(project ""
 				(path "/a75630d2-15a7-42bc-8ce0-7846cbd1da6b/b64ac316-366b-4dad-aacf-d60ea5acbc88/d02d7f80-2025-419a-a5a1-91ce46aa8a95"
-					(reference "R6")
+					(reference "R15")
 					(unit 1)
 				)
@@
 		(dnp no)
 		(fields_autoplaced yes)
-		(property "Reference" "R7"
+		(property "Reference" "R16"
 			(at 182.88 106.6798 90)
 			(effects
@@
 			(project ""
 				(path "/a75630d2-15a7-42bc-8ce0-7846cbd1da6b/b64ac316-366b-4dad-aacf-d60ea5acbc88/d02d7f80-2025-419a-a5a1-91ce46aa8a95"
-					(reference "R7")
-					(unit 1)
-				)
+					(reference "R16")
+					(unit 1)
+				)

Commit message: Addressed DRC warnings and errors.
Connections:
- net GND: now also R15.1, R16.1; no longer R15., R16.
- net at J2.B5 (CC2): now also R15.2; no longer R15.
- net at J2.A5 (CC1): now also R16.2; no longer R16.
Changed lines of the file:
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@@
+	)
+	(junction
+		(at 158.75 50.8)
+		(diameter 0)
+		(color 0 0 0 0)
 	)
 	(junction
@@
 	(wire
 		(pts
-			(xy 154.94 50.8) (xy 165.1 50.8)
+			(xy 154.94 50.8) (xy 158.75 50.8)
 		)
 		(stroke
@@
 	(wire
 		(pts
+			(xy 158.75 50.8) (xy 165.1 50.8)
+		)
+		(stroke
+			(width 0)
+			(type default)
+		)
+	)
+	(wire
+		(pts
 			(xy 147.32 115.57) (xy 152.4 115.57)
 		)
@@
 	)
 	(hierarchical_label "Vin"
-		(shape input)
+		(shape output)
 		(at 165.1 50.8 0)
 		(effects
@@
 		(dnp no)
 		(fields_autoplaced yes)
-		(property "Reference" "#PWR048"
+		(property "Reference" "#PWR48"
 			(at 171.45 137.16 0)
 			(effects
@@
 			(project ""
 				(path "/a75630d2-15a7-42bc-8ce0-7846cbd1da6b/b64ac316-366b-4dad-aacf-d60ea5acbc88/d02d7f80-2025-419a-a5a1-91ce46aa8a95"
-					(reference "#PWR048")
+					(reference "#PWR48")
 					(unit 1)
 				)
@@
 		(dnp no)
 		(fields_autoplaced yes)
-		(property "Reference" "#PWR047"
+		(property "Reference" "#PWR47"
 			(at 152.4 137.16 0)
 			(effects
@@
 			(project ""
 				(path "/a75630d2-15a7-42bc-8ce0-7846cbd1da6b/b64ac316-366b-4dad-aacf-d60ea5acbc88/d02d7f80-2025-419a-a5a1-91ce46aa8a95"
-					(reference "#PWR047")
+					(reference "#PWR47")
 					(unit 1)
 				)
@@
 			)
 		)
-		(pin ""
-		)
-		(pin ""
+		(pin "1"
+		)
+		(pin "2"
 		)
 		(instances
@@
 	)
 	(symbol
-		(lib_name "RC0805FR-075K1L_1")
 		(lib_id "Hourglass_symbol_library:RC0805FR-075K1L")
 		(at 177.8 106.68 90)
@@
 			)
 		)
-		(pin ""
-		)
-		(pin ""
+		(pin "1"
+		)
+		(pin "2"
 		)
 		(instances
@@
 					(unit 1)
 				)
+			)
+		)
+	)
+	(symbol
+		(lib_id "power:PWR_FLAG")
+		(at 158.75 50.8 0)
+		(unit 1)
+		(exclude_from_sim no)
+		(in_bom yes)
+		(on_board yes)
+		(dnp no)
+		(fields_autoplaced yes)
+		(property "Reference" "#FLG1"
+			(at 158.75 48.895 0)
+			(effects
+				(font
+					(size 1.27 1.27)
+				)
+				(hide yes)
+			)
+		)
+		(property "Value" "PWR_FLAG"
+			(at 158.75 45.72 0)
+			(effects
+				(font
+					(size 1.27 1.27)
+				)
+			)
+		)
+		(property "Footprint" ""
+			(at 158.75 50.8 0)
+			(effects
+				(font
+					(size 1.27 1.27)
+				)
+				(hide yes)
+			)
+		)
+		(property "Datasheet" "~"
+			(at 158.75 50.8 0)
+			(effects
+				(font
+					(size 1.27 1.27)
+				)
+				(hide yes)
+			)
+		)
+		(property "Description" "Special symbol for telling ERC where power comes from"
+			(at 158.75 50.8 0)
+			(effects
+				(font
+					(size 1.27 1.27)
+				)
+				(hide yes)
+			)
+		)
+		(pin "1"
+		)
+		(instances
+			(project ""
+				(path "/a75630d2-15a7-42bc-8ce0-7846cbd1da6b/b64ac316-366b-4dad-aacf-d60ea5acbc88/d02d7f80-2025-419a-a5a1-91ce46aa8a95"
+					(reference "#FLG1")
+					(unit 1)
+				)

Commit message: Re-annotated entire schematic.
Parts:
- renumbered R15 to R16, R16 to R17
Other:
- title: (none) -> Hourglass
Changed lines of the file:
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@@
 	(generator_version "9.0")
 	(paper "A4")
+	(title_block
+		(title "Hourglass")
+		(date "2025-04-23")
+		(rev "01")
+	)
 	(text "Placing PD (pull-down)\nresistors to indicate UPSTREAMS device"
 		(exclude_from_sim yes)
@@
 		(dnp no)
 		(fields_autoplaced yes)
-		(property "Reference" "#PWR48"
+		(property "Reference" "#PWR050"
 			(at 171.45 137.16 0)
 			(effects
@@
 			(project ""
 				(path "/a75630d2-15a7-42bc-8ce0-7846cbd1da6b/b64ac316-366b-4dad-aacf-d60ea5acbc88/d02d7f80-2025-419a-a5a1-91ce46aa8a95"
-					(reference "#PWR48")
+					(reference "#PWR050")
 					(unit 1)
 				)
@@
 		(dnp no)
 		(fields_autoplaced yes)
-		(property "Reference" "#PWR47"
+		(property "Reference" "#PWR049"
 			(at 152.4 137.16 0)
 			(effects
@@
 			(project ""
 				(path "/a75630d2-15a7-42bc-8ce0-7846cbd1da6b/b64ac316-366b-4dad-aacf-d60ea5acbc88/d02d7f80-2025-419a-a5a1-91ce46aa8a95"
-					(reference "#PWR47")
+					(reference "#PWR049")
 					(unit 1)
 				)
@@
 		(dnp no)
 		(fields_autoplaced yes)
-		(property "Reference" "R15"
+		(property "Reference" "R16"
 			(at 170.18 106.6798 90)
 			(effects
@@
 			(project ""
 				(path "/a75630d2-15a7-42bc-8ce0-7846cbd1da6b/b64ac316-366b-4dad-aacf-d60ea5acbc88/d02d7f80-2025-419a-a5a1-91ce46aa8a95"
-					(reference "R15")
+					(reference "R16")
 					(unit 1)
 				)
@@
 		(dnp no)
 		(fields_autoplaced yes)
-		(property "Reference" "R16"
+		(property "Reference" "R17"
 			(at 182.88 106.6798 90)
 			(effects
@@
 			(project ""
 				(path "/a75630d2-15a7-42bc-8ce0-7846cbd1da6b/b64ac316-366b-4dad-aacf-d60ea5acbc88/d02d7f80-2025-419a-a5a1-91ce46aa8a95"
-					(reference "R16")
+					(reference "R17")
 					(unit 1)
 				)
@@
 		(dnp no)
 		(fields_autoplaced yes)
-		(property "Reference" "#FLG1"
+		(property "Reference" "#FLG03"
 			(at 158.75 48.895 0)
 			(effects
@@
 			(project ""
 				(path "/a75630d2-15a7-42bc-8ce0-7846cbd1da6b/b64ac316-366b-4dad-aacf-d60ea5acbc88/d02d7f80-2025-419a-a5a1-91ce46aa8a95"
-					(reference "#FLG1")
+					(reference "#FLG03")
 					(unit 1)
 				)
