File: LEDs + Driver.kicad_sch (KiCad schematic)
At the start: 23 parts, among them U2 LP5860

Commit message: Re-annotated entire schematic.
Parts:
- renumbered TP16 to TP10, TP15 to TP11, TP14 to TP12, TP12 to TP14, TP11 to TP15, TP10 to TP16, TP9 to TP17, TP8 to TP18, TP7 to TP19, TP6 to TP20, TP5 to TP21, TP4 to TP22, TP3 to TP23, TP20 to TP6, TP19 to TP7, TP18 to TP8, TP17 to TP9
Other:
- title: (none) -> Hourglass
Changed lines of the file:
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@@
 	(generator_version "9.0")
 	(paper "A4")
+	(title_block
+		(title "Hourglass")
+		(date "2025-04-23")
+		(rev "01")
+	)
 	(rectangle
 		(start 257.81 113.03)
@@
 		(on_board yes)
 		(dnp no)
-		(property "Reference" "TP18"
+		(property "Reference" "TP8"
 			(at 263.9059 72.39 90)
 			(effects
@@
 			(project "Hourglass_PCBA"
 				(path "/a75630d2-15a7-42bc-8ce0-7846cbd1da6b/9c708963-e8cc-42a5-9c83-1e957695e1ca"
-					(reference "TP18")
+					(reference "TP8")
 					(unit 1)
 				)
@@
 		(on_board yes)
 		(dnp no)
-		(property "Reference" "TP7"
+		(property "Reference" "TP19"
 			(at 263.9059 100.33 90)
 			(effects
@@
 			(project "Hourglass_PCBA"
 				(path "/a75630d2-15a7-42bc-8ce0-7846cbd1da6b/9c708963-e8cc-42a5-9c83-1e957695e1ca"
-					(reference "TP7")
+					(reference "TP19")
 					(unit 1)
 				)
@@
 		(dnp no)
 		(fields_autoplaced yes)
-		(property "Reference" "#PWR15"
+		(property "Reference" "#PWR018"
 			(at 100.33 140.97 0)
 			(effects
@@
 			(project ""
 				(path "/a75630d2-15a7-42bc-8ce0-7846cbd1da6b/9c708963-e8cc-42a5-9c83-1e957695e1ca"
-					(reference "#PWR15")
+					(reference "#PWR018")
 					(unit 1)
 				)
@@
 		(on_board yes)
 		(dnp no)
-		(property "Reference" "TP6"
+		(property "Reference" "TP20"
 			(at 263.9059 102.87 90)
 			(effects
@@
 			(project "Hourglass_PCBA"
 				(path "/a75630d2-15a7-42bc-8ce0-7846cbd1da6b/9c708963-e8cc-42a5-9c83-1e957695e1ca"
-					(reference "TP6")
+					(reference "TP20")
 					(unit 1)
 				)
@@
 		(on_board yes)
 		(dnp no)
-		(property "Reference" "TP10"
+		(property "Reference" "TP16"
 			(at 263.9059 92.71 90)
 			(effects
@@
 			(project "Hourglass_PCBA"
 				(path "/a75630d2-15a7-42bc-8ce0-7846cbd1da6b/9c708963-e8cc-42a5-9c83-1e957695e1ca"
-					(reference "TP10")
+					(reference "TP16")
 					(unit 1)
 				)
@@
 		(on_board yes)
 		(dnp no)
-		(property "Reference" "TP11"
+		(property "Reference" "TP15"
 			(at 263.9059 90.17 90)
 			(effects
@@
 			(project "Hourglass_PCBA"
 				(path "/a75630d2-15a7-42bc-8ce0-7846cbd1da6b/9c708963-e8cc-42a5-9c83-1e957695e1ca"
-					(reference "TP11")
+					(reference "TP15")
 					(unit 1)
 				)
@@
 		(dnp no)
 		(fields_autoplaced yes)
-		(property "Reference" "#PWR13"
+		(property "Reference" "#PWR016"
 			(at 55.88 139.7 0)
 			(effects
@@
 			(project "Hourglass_PCBA"
 				(path "/a75630d2-15a7-42bc-8ce0-7846cbd1da6b/9c708963-e8cc-42a5-9c83-1e957695e1ca"
-					(reference "#PWR13")
+					(reference "#PWR016")
 					(unit 1)
 				)
@@
 		(on_board yes)
 		(dnp no)
-		(property "Reference" "TP17"
+		(property "Reference" "TP9"
 			(at 263.9059 74.93 90)
 			(effects
@@
 			(project "Hourglass_PCBA"
 				(path "/a75630d2-15a7-42bc-8ce0-7846cbd1da6b/9c708963-e8cc-42a5-9c83-1e957695e1ca"
-					(reference "TP17")
+					(reference "TP9")
 					(unit 1)
 				)
@@
 		(on_board yes)
 		(dnp no)
-		(property "Reference" "TP20"
+		(property "Reference" "TP6"
 			(at 263.9059 67.31 90)
 			(effects
@@
 			(project "Hourglass_PCBA"
 				(path "/a75630d2-15a7-42bc-8ce0-7846cbd1da6b/9c708963-e8cc-42a5-9c83-1e957695e1ca"
-					(reference "TP20")
+					(reference "TP6")
 					(unit 1)
 				)
@@
 		(on_board yes)
 		(dnp no)
-		(property "Reference" "TP15"
+		(property "Reference" "TP11"
 			(at 263.9059 80.01 90)
 			(effects
@@
 			(project "Hourglass_PCBA"
 				(path "/a75630d2-15a7-42bc-8ce0-7846cbd1da6b/9c708963-e8cc-42a5-9c83-1e957695e1ca"
-					(reference "TP15")
+					(reference "TP11")
 					(unit 1)
 				)
@@
 		(on_board yes)
 		(dnp no)
-		(property "Reference" "#PWR11"
+		(property "Reference" "#PWR013"
 			(at 52.07 26.67 0)
 			(effects
@@
 			(project ""
 				(path "/a75630d2-15a7-42bc-8ce0-7846cbd1da6b/9c708963-e8cc-42a5-9c83-1e957695e1ca"
-					(reference "#PWR11")
+					(reference "#PWR013")
 					(unit 1)
 				)
@@
 		(dnp no)
 		(fields_autoplaced yes)
-		(property "Reference" "#PWR052"
+		(property "Reference" "#PWR015"
 			(at 72.39 67.31 0)
 			(effects
@@
 			(project "Hourglass_PCBA"
 				(path "/a75630d2-15a7-42bc-8ce0-7846cbd1da6b/9c708963-e8cc-42a5-9c83-1e957695e1ca"
-					(reference "#PWR052")
+					(reference "#PWR015")
 					(unit 1)
 				)
@@
 		(dnp no)
 		(fields_autoplaced yes)
-		(property "Reference" "#PWR12"
+		(property "Reference" "#PWR014"
 			(at 44.45 67.31 0)
 			(effects
@@
 			(project ""
 				(path "/a75630d2-15a7-42bc-8ce0-7846cbd1da6b/9c708963-e8cc-42a5-9c83-1e957695e1ca"
-					(reference "#PWR12")
+					(reference "#PWR014")
 					(unit 1)
 				)
@@
 		(on_board yes)
 		(dnp no)
-		(property "Reference" "TP3"
+		(property "Reference" "TP23"
 			(at 263.9059 110.49 90)
 			(effects
@@
 			(project "Hourglass_PCBA"
 				(path "/a75630d2-15a7-42bc-8ce0-7846cbd1da6b/9c708963-e8cc-42a5-9c83-1e957695e1ca"
-					(reference "TP3")
+					(reference "TP23")
 					(unit 1)
 				)
@@
 		(on_board yes)
 		(dnp no)
-		(property "Reference" "TP16"
+		(property "Reference" "TP10"
 			(at 263.9059 77.47 90)
 			(effects
@@
 			(project "Hourglass_PCBA"
 				(path "/a75630d2-15a7-42bc-8ce0-7846cbd1da6b/9c708963-e8cc-42a5-9c83-1e957695e1ca"
-					(reference "TP16")
+					(reference "TP10")
 					(unit 1)
 				)
@@
 		(on_board yes)
 		(dnp no)
-		(property "Reference" "TP8"
+		(property "Reference" "TP18"
 			(at 263.9059 97.79 90)
 			(effects
@@
 			(project "Hourglass_PCBA"
 				(path "/a75630d2-15a7-42bc-8ce0-7846cbd1da6b/9c708963-e8cc-42a5-9c83-1e957695e1ca"
-					(reference "TP8")
+					(reference "TP18")
 					(unit 1)
 				)
@@
 		(on_board yes)
 		(dnp no)
-		(property "Reference" "TP19"
+		(property "Reference" "TP7"
 			(at 263.9059 69.85 90)
 			(effects
@@
 			(project "Hourglass_PCBA"
 				(path "/a75630d2-15a7-42bc-8ce0-7846cbd1da6b/9c708963-e8cc-42a5-9c83-1e957695e1ca"
-					(reference "TP19")
+					(reference "TP7")
 					(unit 1)
 				)
@@
 		(on_board yes)
 		(dnp no)
-		(property "Reference" "TP5"
+		(property "Reference" "TP21"
 			(at 263.9059 105.41 90)
 			(effects
@@
 			(project "Hourglass_PCBA"
 				(path "/a75630d2-15a7-42bc-8ce0-7846cbd1da6b/9c708963-e8cc-42a5-9c83-1e957695e1ca"
-					(reference "TP5")
+					(reference "TP21")
 					(unit 1)
 				)
@@
 		(on_board yes)
 		(dnp no)
-		(property "Reference" "TP4"
+		(property "Reference" "TP22"
 			(at 263.9059 107.95 90)
 			(effects
@@
 			(project "Hourglass_PCBA"
 				(path "/a75630d2-15a7-42bc-8ce0-7846cbd1da6b/9c708963-e8cc-42a5-9c83-1e957695e1ca"
-					(reference "TP4")
+					(reference "TP22")
 					(unit 1)
 				)
@@
 		(dnp no)
 		(fields_autoplaced yes)
-		(property "Reference" "#PWR14"
+		(property "Reference" "#PWR017"
 			(at 62.23 139.7 0)
 			(effects
@@
 			(project "Hourglass_PCBA"
 				(path "/a75630d2-15a7-42bc-8ce0-7846cbd1da6b/9c708963-e8cc-42a5-9c83-1e957695e1ca"
-					(reference "#PWR14")
+					(reference "#PWR017")
 					(unit 1)
 				)
@@
 		(on_board yes)
 		(dnp no)
-		(property "Reference" "TP9"
+		(property "Reference" "TP17"
 			(at 263.9059 95.25 90)
 			(effects
@@
 			(project "Hourglass_PCBA"
 				(path "/a75630d2-15a7-42bc-8ce0-7846cbd1da6b/9c708963-e8cc-42a5-9c83-1e957695e1ca"
-					(reference "TP9")
+					(reference "TP17")
 					(unit 1)
 				)
@@
 		(on_board yes)
 		(dnp no)
-		(property "Reference" "TP12"
+		(property "Reference" "TP14"
 			(at 263.9059 87.63 90)
 			(effects
@@
 			(project "Hourglass_PCBA"
 				(path "/a75630d2-15a7-42bc-8ce0-7846cbd1da6b/9c708963-e8cc-42a5-9c83-1e957695e1ca"
-					(reference "TP12")
+					(reference "TP14")
 					(unit 1)
 				)
@@
 		(on_board yes)
 		(dnp no)
-		(property "Reference" "TP14"
+		(property "Reference" "TP12"
 			(at 263.9059 82.55 90)
 			(effects
@@
 			(project "Hourglass_PCBA"
 				(path "/a75630d2-15a7-42bc-8ce0-7846cbd1da6b/9c708963-e8cc-42a5-9c83-1e957695e1ca"
-					(reference "TP14")
+					(reference "TP12")
 					(unit 1)
 				)

Commit message: Updated the 3D models
Other:
- note added: "TPs currently not inclucded due to space"
Changed lines of the file:
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@@
 		)
 	)
+	(text "TPs currently not \ninclucded due to space 	"
+		(exclude_from_sim yes)
+		(at 258.826 116.078 0)
+		(effects
+			(font
+				(size 1.27 1.27)
+			)
+			(justify left)
+		)
+	)
 	(text "Place CAPs ACAP to U2\n"
 		(exclude_from_sim yes)
@@
 		(exclude_from_sim no)
 		(in_bom yes)
-		(on_board yes)
+		(on_board no)
 		(dnp no)
 		(property "Reference" "TP8"
@@
 		(exclude_from_sim no)
 		(in_bom yes)
-		(on_board yes)
+		(on_board no)
 		(dnp no)
 		(property "Reference" "TP19"
@@
 		(exclude_from_sim no)
 		(in_bom yes)
-		(on_board yes)
+		(on_board no)
 		(dnp no)
 		(property "Reference" "TP20"
@@
 		(exclude_from_sim no)
 		(in_bom yes)
-		(on_board yes)
+		(on_board no)
 		(dnp no)
 		(property "Reference" "TP16"
@@
 		(exclude_from_sim no)
 		(in_bom yes)
-		(on_board yes)
+		(on_board no)
 		(dnp no)
 		(property "Reference" "TP15"
@@
 		(exclude_from_sim no)
 		(in_bom yes)
-		(on_board yes)
+		(on_board no)
 		(dnp no)
 		(property "Reference" "TP9"
@@
 		(exclude_from_sim no)
 		(in_bom yes)
-		(on_board yes)
+		(on_board no)
 		(dnp no)
 		(property "Reference" "TP6"
@@
 		(exclude_from_sim no)
 		(in_bom yes)
-		(on_board yes)
+		(on_board no)
 		(dnp no)
 		(property "Reference" "TP11"
@@
 		(exclude_from_sim no)
 		(in_bom yes)
-		(on_board yes)
+		(on_board no)
 		(dnp no)
 		(property "Reference" "TP23"
@@
 		(exclude_from_sim no)
 		(in_bom yes)
-		(on_board yes)
+		(on_board no)
 		(dnp no)
 		(property "Reference" "TP10"
@@
 		(exclude_from_sim no)
 		(in_bom yes)
-		(on_board yes)
+		(on_board no)
 		(dnp no)
 		(property "Reference" "TP18"
@@
 		(exclude_from_sim no)
 		(in_bom yes)
-		(on_board yes)
+		(on_board no)
 		(dnp no)
 		(property "Reference" "TP7"
@@
 		(exclude_from_sim no)
 		(in_bom yes)
-		(on_board yes)
+		(on_board no)
 		(dnp no)
 		(property "Reference" "TP13"
@@
 		(exclude_from_sim no)
 		(in_bom yes)
-		(on_board yes)
+		(on_board no)
 		(dnp no)
 		(property "Reference" "TP21"
@@
 		(exclude_from_sim no)
 		(in_bom yes)
-		(on_board yes)
+		(on_board no)
 		(dnp no)
 		(property "Reference" "TP22"
@@
 		(exclude_from_sim no)
 		(in_bom yes)
-		(on_board yes)
+		(on_board no)
 		(dnp no)
 		(property "Reference" "TP17"
@@
 		(exclude_from_sim no)
 		(in_bom yes)
-		(on_board yes)
+		(on_board no)
 		(dnp no)
 		(property "Reference" "TP14"
@@
 		(exclude_from_sim no)
 		(in_bom yes)
-		(on_board yes)
+		(on_board no)
 		(dnp no)
 		(property "Reference" "TP12"
