File: Hourglass_PCBA.kicad_pcb (KiCad board)
At the start: 4 copper layers, 40.9 x 87.5 mm, 134 parts, among them J1 B2B-PH-SM4-TBLFSN, J2 UJ31-CH-G2-SMT-TR, J3 009159010061911, SW1 KMR221NGLFS, U1 STM32L432KCUx, U2 LP5860, U3 LSM6DSOXTR, U4 MCP1727T-3302E/SN, U5 BQ25185DLHR

Commit message: Progress commit
Parts:
- moved FB1 22.8 mm to (205.1, 159.9), turned to 180 degrees
- moved R1 20.5 mm to (207.5, 162.9), turned to 180 degrees
- moved R4 20.1 mm to (190.9, 165.1)
- moved C4 19.6 mm to (203.0, 159.5), turned to 90 degrees
- moved C5 18.1 mm to (201.6, 159.5), turned to 90 degrees
- moved TP36 17.8 mm to (223.4, 163.0)
- moved TP2 16.8 mm to (222.0, 166.9)
- moved R6 16.0 mm to (204.9, 177.8), turned to 180 degrees
- moved TP3 14.2 mm to (220.9, 170.1)
- moved TP30 14.1 mm to (224.2, 177.6)
- moved C6 13.9 mm to (212.9, 163.0)
- moved C1 12.8 mm to (193.4, 160.2), turned to 90 degrees
- moved TP4 12.5 mm to (215.7, 183.3)
- moved C11 11.7 mm to (197.1, 174.1), turned to 90 degrees
- moved C2 11.7 mm to (194.8, 160.2), turned to 90 degrees
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Routing:
- net /LED Driver +  LEDs/CS0: track 4.61 -> 42.9 mm, vias 0 -> 5
- net GND: track 8.56 -> 45.9 mm, vias 19 -> 37
- net /MCU/NRST: track 0.00 -> 26.0 mm
- net /LED Driver +  LEDs/CS2: track 0.00 -> 25.1 mm, vias 0 -> 5
- net /LED Driver +  LEDs/CS1: track 0.00 -> 20.4 mm, vias 0 -> 5
- net /LED Driver +  LEDs/VSYNC: track 3.71 -> 17.5 mm, vias 0 -> 2
- net /LSM6DSOX 6-Axis IMU/LSM6DSOX_INT1: track 0.00 -> 12.2 mm, vias 0 -> 2
- net /LED Driver +  LEDs/CS12: track 5.56 -> 16.8 mm, vias 1 -> 4
- net /LED Driver +  LEDs/CS13: track 6.21 -> 17.4 mm, vias 1 -> 4
- net +3V3: track 4.64 -> 15.3 mm
- net /LED Driver +  LEDs/CS5: track 0.00 -> 9.06 mm, vias 0 -> 4
- net /LED Driver +  LEDs/CS8: track 0.00 -> 8.22 mm, vias 0 -> 4
- net /LED Driver +  LEDs/CS7: track 0.00 -> 7.12 mm, vias 0 -> 4
- net /LED Driver +  LEDs/CS4: track 0.00 -> 6.33 mm, vias 0 -> 4
- net /LED Driver +  LEDs/CS14: track 5.82 -> 12.1 mm, vias 1 -> 4
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